File: PMSM_Driver/PMSM_Driver.kicad_pcb (KiCad board)
At the start: 2 copper layers, 244.9 x 138.4 mm, 231 parts, among them J1 Screw_Terminal_01x03, J10 AFBR-2624Z, J11 AFBR-2624Z, J12 AFBR-2624Z, J13 AFBR-2624Z, J14 AFBR-2624Z, J15 AFBR-2624Z, J16 AFBR-2624Z, J17 AFBR-1624Z, J18 AFBR-1624Z, J2 AFBR-2624Z, J3 Screw_Terminal_01x02, J4 Screw_Terminal_01x02, J5 AFBR-1624Z, J6 AFBR-2624Z, J7 AFBR-2624Z, J8 AFBR-2624Z, J9 AFBR-2624Z, Q1 BC846, Q10 BC846, Q11 RGCL60TK60, Q12 RGCL60TK60, Q13 RGCL60TK60, Q14 RGCL60TK60, Q15 BC846, Q16 RGCL60TK60, Q17 RGCL60TK60, Q18 RGCL60TK60, Q19 RGCL60TK60, Q2 BC846, Q20 BC846, Q21 BC846, Q22 BC846, Q23 BC846, Q24 BC846, Q3 BC846, Q4 BC846, Q5 RGCL60TK60, Q6 RGCL60TK60, Q7 RGCL60TK60, Q8 RGCL60TK60, Q9 BC846, U1 74LVC1G04, U10 HCPL-3120, U11 HCPL-3120, U12 HCPL-3120, U13 74LVC1G04, U14 74LVC1G04, U15 74LVC1G04, U16 MGJ2D051515SC, U17 MGJ2D051515SC, U18 MGJ2D051515SC, U19 HCPL-3120, U2 MGJ2D051515SC, U20 HCPL-3120, U21 HCPL-3120, U22 74LVC1G04, U23 74LVC1G04, U24 74LVC1G04, U25 MGJ2D051515SC, U26 MGJ2D051515SC, U27 MGJ2D051515SC, U28 HCPL-3120, U29 HCPL-3120, U3 HCPL-3120, U30 HCPL-3120, U31 74LVC1G04, U32 74LVC1G04, U33 MGJ2D051515SC, U34 MGJ2D051515SC, U35 HCPL-3120, U36 HCPL-3120, U37 VS-E5TH3006S2L-M3, U38 VS-E5TH3006S2L-M3, U39 VS-E5TH3006S2L-M3, U4 74LVC1G04, U40 VS-E5TH3006S2L-M3, U41 VS-E5TH3006S2L-M3, U42 VS-E5TH3006S2L-M3, U43 VS-E5TH3006S2L-M3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

Commit message: update on PCB layout
Parts:
- J1: value Screw_Terminal_01x03 -> 1714984; footprint TerminalBlock_Phoenix:TerminalBlock_Phoenix_MKDS-1,5-3-5.08_1x03_P5.08mm_Horizontal -> FYP_Components:CONN_1714984_PXC
- J3: value Screw_Terminal_01x02 -> 1714971; footprint FYP_Components:8PCV-02-006 -> FYP_Components:CONN_1714971_PXC
- J4: value Screw_Terminal_01x02 -> 1714971; footprint TerminalBlock_Phoenix:TerminalBlock_Phoenix_MKDS-1,5-2-5.08_1x02_P5.08mm_Horizontal -> FYP_Components:CONN_1714971_PXC
- moved J16 30.0 mm to (186.5, 54.0)
- moved J13 15.1 mm to (201.7, 54.0)
- moved J10 15.0 mm to (216.7, 53.8)
- moved J3 13.5 mm to (62.1, 112.3)
- moved U42 7.10 mm to (232.9, 144.7)
- moved U41 7.08 mm to (233.1, 83.2)
- moved U40 6.85 mm to (164.6, 144.3)
- moved U39 6.51 mm to (164.7, 83.1)
- moved J4 6.04 mm to (62.1, 63.8)
- moved C14 5.09 mm to (80.1, 105.5)
- moved R4 5.09 mm to (91.0, 105.6)
- moved R5 5.09 mm to (91.5, 126.7)
- moved C15 5.09 mm to (80.2, 126.9)
- moved C1 4.63 mm to (71.4, 60.6)
- moved C4 4.63 mm to (69.2, 63.2)
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Connections:
- C10 pad 2: Net-(U2-0V) -> /C1_E
- C11 pad 1: Net-(U2-0V) -> /C1_E
- C12 pad 2: Net-(U2-0V) -> /C1_E
- C13 pad 1: Net-(U2-0V) -> /C1_E
- C16 pad 2: Net-(U7-0V) -> /B1_E
- C17 pad 1: Net-(U7-0V) -> /B1_E
- C18 pad 2: Net-(U8-0V) -> /A1_E
- C19 pad 1: Net-(U8-0V) -> /A1_E
- C20 pad 2: Net-(U9-0V) -> ic_out
- C21 pad 1: Net-(U9-0V) -> ic_out
- C21 pad 2: ic_out -> /-15V_C2
- C22 pad 2: Net-(U7-0V) -> /B1_E
- C23 pad 1: Net-(U7-0V) -> /B1_E
- C24 pad 2: Net-(U8-0V) -> /A1_E
- C25 pad 1: Net-(U8-0V) -> /A1_E
- C26 pad 2: Net-(U9-0V) -> ic_out
- C27 pad 1: Net-(U9-0V) -> ic_out
- C27 pad 2: ic_out -> /-15V_C2
- C28 pad 2: Net-(U7-0V) -> /B1_E
- C29 pad 1: Net-(U7-0V) -> /B1_E
- C30 pad 2: Net-(U8-0V) -> /A1_E
- C31 pad 1: Net-(U8-0V) -> /A1_E
- C32 pad 2: Net-(U9-0V) -> ic_out
- C33 pad 1: Net-(U9-0V) -> ic_out
- C33 pad 2: ic_out -> /-15V_C2
- C34 pad 2: Net-(U16-0V) -> ib_out
- C35 pad 1: Net-(U16-0V) -> ib_out
- C35 pad 2: ib_out -> /-15V_B2
- C36 pad 2: Net-(U17-0V) -> ia_out
- C37 pad 1: Net-(U17-0V) -> ia_out
- C37 pad 2: ia_out -> /-15V_A2
- C38 pad 2: Net-(U16-0V) -> ib_out
- C39 pad 1: Net-(U16-0V) -> ib_out
- C39 pad 2: ib_out -> /-15V_B2
- C40 pad 2: Net-(U17-0V) -> ia_out
- C41 pad 1: Net-(U17-0V) -> ia_out
- C41 pad 2: ia_out -> /-15V_A2
- C42 pad 2: Net-(U18-0V) -> /C3_E
- C43 pad 1: Net-(U18-0V) -> /C3_E
- C44 pad 2: Net-(U16-0V) -> ib_out
- C45 pad 1: Net-(U16-0V) -> ib_out
- C45 pad 2: ib_out -> /-15V_B2
- C46 pad 2: Net-(U17-0V) -> ia_out
- C47 pad 1: Net-(U17-0V) -> ia_out
- C47 pad 2: ia_out -> /-15V_A2
- C48 pad 2: Net-(U18-0V) -> /C3_E
- C49 pad 1: Net-(U18-0V) -> /C3_E
- C50 pad 2: Net-(U18-0V) -> /C3_E
- C51 pad 1: Net-(U18-0V) -> /C3_E
- C52 pad 2: Net-(U25-0V) -> /B3_E
- C53 pad 1: Net-(U25-0V) -> /B3_E
- C54 pad 2: Net-(U26-0V) -> /A3_E
- C55 pad 1: Net-(U26-0V) -> /A3_E
- C56 pad 2: Net-(U27-0V) -> -BATT
- C57 pad 1: Net-(U27-0V) -> -BATT
- C57 pad 2: -BATT -> /-15V_C4
- C58 pad 2: Net-(U25-0V) -> /B3_E
- C59 pad 1: Net-(U25-0V) -> /B3_E
- C60 pad 2: Net-(U26-0V) -> /A3_E
- C61 pad 1: Net-(U26-0V) -> /A3_E
- C62 pad 2: Net-(U27-0V) -> -BATT
- C63 pad 1: Net-(U27-0V) -> -BATT
- C63 pad 2: -BATT -> /-15V_C4
- C64 pad 2: Net-(U25-0V) -> /B3_E
- C65 pad 1: Net-(U25-0V) -> /B3_E
- C66 pad 2: Net-(U26-0V) -> /A3_E
- C67 pad 1: Net-(U26-0V) -> /A3_E
- C68 pad 2: Net-(U27-0V) -> -BATT
- C69 pad 1: Net-(U27-0V) -> -BATT
- C69 pad 2: -BATT -> /-15V_C4
- C7 pad 2: Net-(U2-0V) -> /C1_E
- C70 pad 2: Net-(U33-0V) -> -BATT
- C71 pad 1: Net-(U33-0V) -> -BATT
- C71 pad 2: -BATT -> /-15V_B4
- C72 pad 2: Net-(U34-0V) -> -BATT
- C73 pad 1: Net-(U34-0V) -> -BATT
- C73 pad 2: -BATT -> /-15V_A4
- C74 pad 2: Net-(U33-0V) -> -BATT
- C75 pad 1: Net-(U33-0V) -> -BATT
- C75 pad 2: -BATT -> /-15V_B4
- C76 pad 2: Net-(U34-0V) -> -BATT
- C77 pad 1: Net-(U34-0V) -> -BATT
- C77 pad 2: -BATT -> /-15V_A4
- C78 pad 2: Net-(U33-0V) -> -BATT
- C79 pad 1: Net-(U33-0V) -> -BATT
- C79 pad 2: -BATT -> /-15V_B4
- C8 pad 1: Net-(U2-0V) -> /C1_E
- C80 pad 2: Net-(U34-0V) -> -BATT
- C81 pad 1: Net-(U34-0V) -> -BATT
- C81 pad 2: -BATT -> /-15V_A4
- Q1 pad 2: GNDD -> GND
- Q10 pad 2: GNDD -> GND
- Q11 pad 3: /-15V_B1 -> /B1_E
- Q12 pad 2: /-15V_B1 -> /B1_E
- Q13 pad 3: /-15V_B3 -> /B3_E
- Q14 pad 2: /-15V_B3 -> /B3_E
- Q15 pad 2: GNDD -> GND
- Q16 pad 3: /-15V_C1 -> /C1_E
- Q17 pad 2: /-15V_C1 -> /C1_E
- Q18 pad 3: /-15V_C3 -> /C3_E
- Q19 pad 2: /-15V_C3 -> /C3_E
- Q2 pad 2: GNDD -> GND
- Q20 pad 2: GNDD -> GND
- Q21 pad 2: GNDD -> GND
- Q22 pad 2: GNDD -> GND
- Q23 pad 2: GNDD -> GND
- Q24 pad 2: GNDD -> GND
- Q3 pad 2: GNDD -> GND
- Q4 pad 2: GNDD -> GND
- Q5 pad 3: /-15V_A1 -> /A1_E
- Q6 pad 2: /-15V_A1 -> /A1_E
- Q7 pad 3: /-15V_A3 -> /A3_E
- Q8 pad 2: /-15V_A3 -> /A3_E
- Q9 pad 2: GNDD -> GND
- U10 pad 3: GNDD -> GND
- U11 pad 3: GNDD -> GND
- U12 pad 3: GNDD -> GND
- U12 pad 5: ic_out -> /-15V_C2
- U16 pad 5: ib_out -> /-15V_B2
- U16 pad 6: Net-(U16-0V) -> ib_out
- U17 pad 5: ia_out -> /-15V_A2
- U17 pad 6: Net-(U17-0V) -> ia_out
- U18 pad 6: Net-(U18-0V) -> /C3_E
- U19 pad 3: GNDD -> GND
- U19 pad 5: ib_out -> /-15V_B2
- U2 pad 6: Net-(U2-0V) -> /C1_E
- U20 pad 3: GNDD -> GND
- U20 pad 5: ia_out -> /-15V_A2
- U21 pad 3: GNDD -> GND
- U25 pad 6: Net-(U25-0V) -> /B3_E
- U26 pad 6: Net-(U26-0V) -> /A3_E
- U27 pad 5: -BATT -> /-15V_C4
- U27 pad 6: Net-(U27-0V) -> -BATT
- U28 pad 3: GNDD -> GND
- U29 pad 3: GNDD -> GND
- U3 pad 3: GNDD -> GND
- U30 pad 3: GNDD -> GND
- U30 pad 5: -BATT -> /-15V_C4
- U33 pad 5: -BATT -> /-15V_B4
- U33 pad 6: Net-(U33-0V) -> -BATT
- U34 pad 5: -BATT -> /-15V_A4
- U34 pad 6: Net-(U34-0V) -> -BATT
- U35 pad 3: GNDD -> GND
- U35 pad 5: -BATT -> /-15V_B4
- U36 pad 3: GNDD -> GND
- U36 pad 5: -BATT -> /-15V_A4
- U37 pad 2: /-15V_A1 -> /A1_E
- U38 pad 1: /-15V_A3 -> /A3_E
- U38 pad 3: /-15V_A3 -> /A3_E
- U39 pad 2: /-15V_B1 -> /B1_E
- U40 pad 1: /-15V_B3 -> /B3_E
- U40 pad 3: /-15V_B3 -> /B3_E
- U41 pad 2: /-15V_C1 -> /C1_E
- U42 pad 1: /-15V_C3 -> /C3_E
- U42 pad 3: /-15V_C3 -> /C3_E
- U43 pad 1: /-15V_A1 -> /A1_E
- U43 pad 3: /-15V_A1 -> /A1_E
- U44 pad 2: /-15V_A1 -> /A1_E
- U45 pad 1: /-15V_A3 -> /A3_E
- U45 pad 3: /-15V_A3 -> /A3_E
- U46 pad 2: /-15V_A3 -> /A3_E
- U47 pad 1: /-15V_B1 -> /B1_E
- U47 pad 3: /-15V_B1 -> /B1_E
- U48 pad 2: /-15V_B1 -> /B1_E
- U49 pad 1: /-15V_B3 -> /B3_E
- U49 pad 3: /-15V_B3 -> /B3_E
- U50 pad 2: /-15V_B3 -> /B3_E
- U51 pad 1: /-15V_C1 -> /C1_E
- U51 pad 3: /-15V_C1 -> /C1_E
- U52 pad 2: /-15V_C1 -> /C1_E
- U53 pad 1: /-15V_C3 -> /C3_E
- U53 pad 3: /-15V_C3 -> /C3_E
- U54 pad 2: /-15V_C3 -> /C3_E
- U7 pad 6: Net-(U7-0V) -> /B1_E
- U8 pad 6: Net-(U8-0V) -> /A1_E
- U9 pad 5: ic_out -> /-15V_C2
- U9 pad 6: Net-(U9-0V) -> ic_out
Routing:
- net +5V: track 0.00 -> 371.4 mm
- net ia_signal: track 0.00 -> 148.1 mm, vias 0 -> 2
- net Net-(J16-Data_Out): track 0.00 -> 139.8 mm, vias 0 -> 1
- net Net-(J15-Data_Out): track 0.00 -> 136.7 mm, vias 0 -> 1
- net Net-(J14-Data_Out): track 0.00 -> 132.1 mm, vias 0 -> 1
- net Net-(J13-Data_Out): track 0.00 -> 104.3 mm, vias 0 -> 1
- net a_out: track 0.00 -> 103.1 mm, vias 0 -> 1
- net Net-(J12-Data_Out): track 0.00 -> 100.3 mm, vias 0 -> 1
- net Net-(J11-Data_Out): track 0.00 -> 95.9 mm, vias 0 -> 1
- net /A1_E: track 0.00 -> 94.8 mm, vias 0 -> 2
- net c_out: track 0.00 -> 86.8 mm, vias 0 -> 1
- net Net-(J10-Data_Out): track 0.00 -> 67.4 mm, vias 0 -> 1
- net GND: track 0.00 -> 65.7 mm, vias 0 -> 5
- net b_out: track 0.00 -> 64.2 mm, vias 0 -> 1
- net Net-(J9-Data_Out): track 0.00 -> 64.0 mm, vias 0 -> 1
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- added copper zone on F.Cu, net +BATT
- added copper zone on In1.Cu, net +BATT
- added copper zone on In2.Cu, net -BATT
- added copper zone on F.Cu, net /A1
- added copper zone on F.Cu, net /A1_E
- added copper zone on In1.Cu, net /A2
- added copper zone on B.Cu, net GND
Other:
- board size 244.9 x 138.4 mm -> 244.9 x 140.1 mm
- copper layers 2 -> 4
- board text added: "A1"
- board text added: "A2"
- board text added: "A3"
- board text added: "A4"
- board text added: "B1"
- board text added: "B2"
- board text added: "B3"
- board text added: "B4"
- board text added: "C1"
- board text added: "C2"
- board text added: "C3"
- board text added: "C4"
- board text added: "IA"
- board text added: "IB"
- board text added: "IC"

Commit message: updated the PCB layout
Parts:
- moved U42 17.5 mm to (233.3, 127.2)
- moved U38 17.4 mm to (102.4, 127.2)
- moved U40 17.1 mm to (165.3, 127.2)
- moved U39 1.35 mm to (165.5, 84.2)
- moved U37 0.85 mm to (99.8, 84.1)
- moved U51 0.62 mm to (280.4, 72.1)
- moved U41 0.61 mm to (232.9, 83.8)
- moved U47 0.60 mm to (211.9, 72.0)
- moved U43 0.56 mm to (143.6, 72.0)
Routing:
- net +5V: track 371.4 -> 0.11 mm
- net /B1_E: track 0.00 -> 73.7 mm, vias 0 -> 1
- net /A3_E: track 43.7 -> 111.6 mm, vias 0 -> 1
- net -BATT: track 37.1 -> 81.0 mm
- net /C1_E: track 0.00 -> 32.5 mm, vias 0 -> 1
- net /-15V_B1: track 0.00 -> 32.1 mm
- net ia_out: track 62.6 -> 93.1 mm
- net /-15V_A4: track 0.00 -> 30.4 mm
- net /-15V_A3: track 9.83 -> 31.5 mm
- net /+15V_B1: track 0.00 -> 21.2 mm
- net /+15V_A4: track 0.00 -> 20.4 mm
- net GND: track 65.7 -> 84.7 mm, vias 5 -> 11
- net /A1_E: track 94.8 -> 111.2 mm
- net +BATT: track 37.1 -> 52.5 mm
- net ib_out: track 0.00 -> 11.6 mm
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- added copper zone on F.Cu, net +5V
- added copper zone on F.Cu, net /A2
- added copper zone on F.Cu, net /A3
- added copper zone on F.Cu, net /A4
- added copper zone on In2.Cu, net GNDREF
- removed copper zone on F.Cu, net +BATT
- removed copper zone on F.Cu, net /A1_E
- removed copper zone on In1.Cu, net /A2

Commit message: complete the PCB layout
Routing:
- net /C3_E: track 0.00 -> 117.7 mm, vias 0 -> 1
- net /B3_E: track 5.08 -> 116.4 mm, vias 0 -> 1
- net GNDREF: track 35.1 -> 140.7 mm, vias 0 -> 25
- net ic_out: track 0.00 -> 97.1 mm, vias 0 -> 1
- net ib_signal: track 6.71 -> 95.6 mm, vias 0 -> 2
- net ib_out: track 11.6 -> 97.1 mm, vias 0 -> 1
- net /C1_E: track 32.5 -> 113.8 mm
- net -BATT: track 81.0 -> 155.9 mm
- net ic_signal: track 6.55 -> 65.7 mm, vias 0 -> 2
- net GND: track 84.7 -> 139.0 mm, vias 11 -> 27
- net /B1_E: track 73.7 -> 115.3 mm
- net /-15V_C4: track 0.00 -> 31.9 mm
- net /-15V_C1: track 0.00 -> 31.9 mm
- net /-15V_B3: track 0.00 -> 31.7 mm
- net /-15V_C2: track 0.00 -> 31.5 mm
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- removed copper zone on F.Cu, net /A1
- removed copper zone on F.Cu, net /A2
- removed copper zone on F.Cu, net /A3
- removed copper zone on F.Cu, net /A4

Commit message: add single buffers to signal output, update layout
Parts:
- added U58: SN74LV1T34DBV, Package_TO_SOT_SMD:SOT-23-5, F.Cu at (144.3, 111.1)
- added U59: SN74LV1T34DBV, Package_TO_SOT_SMD:SOT-23-5, F.Cu at (212.5, 111.5)
- added U60: SN74LV1T34DBV, Package_TO_SOT_SMD:SOT-23-5, F.Cu at (281.1, 111.1)
- moved C9 14.0 mm to (70.6, 72.2)
- moved C6 9.40 mm to (70.6, 69.9)
- moved C2 5.87 mm to (70.5, 60.2)
- moved C5 4.30 mm to (70.6, 67.5)
- moved C3 3.43 mm to (70.6, 62.6)
- moved C1 2.92 mm to (70.5, 57.8)
- moved H2 2.50 mm to (290.2, 45.1)
- moved C4 2.31 mm to (70.6, 65.1)
- moved H1 2.26 mm to (58.9, 45.2)
- moved U50 1.09 mm to (211.3, 159.6)
- moved H4 0.54 mm to (289.7, 175.4)
Connections:
- C82 pad 1: ia_signal -> Net-(U55-VIOUT)
- C83 pad 1: ib_signal -> Net-(U56-VIOUT)
- C84 pad 1: ic_signal -> Net-(U57-VIOUT)
- U55 pad 7: ia_signal -> Net-(U55-VIOUT)
- U56 pad 7: ib_signal -> Net-(U56-VIOUT)
- U57 pad 7: ic_signal -> Net-(U57-VIOUT)
Routing:
- net +5V: track 0.11 -> 33.2 mm
- net -BATT: track 155.9 -> 178.1 mm
- net ic_signal: track 65.7 -> 57.1 mm
- net ib_signal: track 95.6 -> 88.3 mm
- net ia_signal: track 143.8 -> 137.1 mm
- net Net-(U55-VIOUT): track 0.00 -> 6.09 mm
- net Net-(U56-VIOUT): track 0.00 -> 5.94 mm
- net Net-(U57-VIOUT): track 0.00 -> 5.79 mm
- net GND: track 139.0 -> 137.1 mm
- net Net-(J13-Data_Out): track 104.3 -> 105.7 mm
- net Net-(J6-Data_Out): track 25.0 -> 26.0 mm
- net /-15V_A4: track 30.4 -> 31.1 mm
- net /A1_E: vias 2 -> 1
Other:
- board size 244.9 x 140.1 mm -> 244.8 x 144.1 mm
- board text added: "+BATT"
- board text added: "-BATT"
- board text added: "A_OUT"
- board text added: "B_OUT"
- board text added: "C_OUT"
- board text added: "GNDREF"
