File: PMSM_Driver/PMSM_Driver.kicad_pcb (KiCad board)
At the start: 4 copper layers, 265.6 x 144 mm, 276 parts, among them J1 2606-1101, J10 AFBR-2624Z, J11 AFBR-2624Z, J12 AFBR-2624Z, J13 AFBR-2624Z, J14 AFBR-2624Z, J15 AFBR-2624Z, J16 AFBR-2624Z, J17 2606-1101, J18 2606-1101, J2 AFBR-2624Z, J3 1714971, J4 1714971, J5 1827907, J6 AFBR-2624Z, J7 AFBR-2624Z, J8 AFBR-2624Z, J9 AFBR-2624Z, Q1 BC846, Q10 BC846, Q11 RGCL60TK60, Q12 RGCL60TK60, Q13 RGCL60TK60, Q14 RGCL60TK60, Q15 BC846, Q16 RGCL60TK60, Q17 RGCL60TK60, Q18 RGCL60TK60, Q19 RGCL60TK60, Q2 BC846, Q20 BC846, Q21 BC846, Q22 BC846, Q23 BC846, Q24 BC846, Q3 BC846, Q4 BC846, Q5 RGCL60TK60, Q6 RGCL60TK60, Q7 RGCL60TK60, Q8 RGCL60TK60, Q9 BC846, U1 74LVC1G04, U10 HCPL-3120, U11 HCPL-3120, U12 HCPL-3120, U13 74LVC1G04, U14 74LVC1G04, U15 74LVC1G04, U16 MGJ2D051515SC, U17 MGJ2D051515SC, U18 MGJ2D051515SC, U19 HCPL-3120, U2 MGJ2D051515SC, U20 HCPL-3120, U21 HCPL-3120, U22 74LVC1G04, U23 74LVC1G04, U24 74LVC1G04, U25 MGJ2D051515SC, U26 MGJ2D051515SC, U27 MGJ2D051515SC, U28 HCPL-3120, U29 HCPL-3120, U3 HCPL-3120, U30 HCPL-3120, U31 74LVC1G04, U32 74LVC1G04, U33 MGJ2D051515SC, U34 MGJ2D051515SC, U35 HCPL-3120, U36 HCPL-3120, U37 VS-E5TH3006S2L-M3, U38 VS-E5TH3006S2L-M3, U39 VS-E5TH3006S2L-M3, U4 74LVC1G04, U40 VS-E5TH3006S2L-M3, U41 VS-E5TH3006S2L-M3, U42 VS-E5TH3006S2L-M3, U43 VS-E5TH3006S2L-M3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

Commit message: Final Version 1 Update
Parts:
- added C85: 0.1u, Capacitor_SMD:C_1206_3216Metric, B.Cu at (245.7, 50.9)
- added C86: 0.1u, Capacitor_SMD:C_1206_3216Metric, B.Cu at (230.4, 50.9)
- added C87: 0.1u, Capacitor_SMD:C_1206_3216Metric, B.Cu at (214.8, 50.8)
- added C88: 0.1u, Capacitor_SMD:C_1206_3216Metric, B.Cu at (199.0, 50.9)
- added C89: 0.1u, Capacitor_SMD:C_1206_3216Metric, B.Cu at (183.5, 50.8)
- added C90: 1u, Capacitor_SMD:C_1206_3216Metric, B.Cu at (55.9, 69.0)
- added C91: 1u, Capacitor_SMD:C_1206_3216Metric, B.Cu at (58.3, 69.0)
- added C92: 1u, Capacitor_SMD:C_1206_3216Metric, B.Cu at (62.1, 69.0)
- added C93: 1u, Capacitor_SMD:C_1206_3216Metric, B.Cu at (64.5, 69.0)
- added C94: 1u, Capacitor_SMD:C_1206_3216Metric, B.Cu at (67.0, 69.0)
- added C95: 1n, Capacitor_SMD:C_1206_3216Metric, F.Cu at (152.7, 116.3)
- added C96: 1n, Capacitor_SMD:C_1206_3216Metric, F.Cu at (221.8, 116.5)
- added C97: 1n, Capacitor_SMD:C_1206_3216Metric, F.Cu at (290.7, 115.3)
- C1, C2, C4, C6, C9: value 1u -> 0.1u; footprint Capacitor_SMD:C_0402_1005Metric -> Capacitor_SMD:C_1206_3216Metric
- C10, C11, C12, C13, C16, C17, C18, C19, C20, C21, C22, C23, C24, C25, C26, C27, C28, C29, C30, C31, C32, C33, C34, C35, C36, C37, C38, C39, C40, C41, C42, C43, C44, C45, C46, C47, C48, C49, C50, C51, C52, C53, C54, C55, C56, C57, C58, C59, C60, C61, C62, C63, C64, C65, C66, C67, C68, C69, C7, C70, C71, C72, C73, C74, C75, C76, C77, C78, C79, C8, C80, C81: footprint Capacitor_SMD:C_0402_1005Metric -> Capacitor_SMD:C_1206_3216Metric; moved to B.Cu
- C3, C5: footprint Capacitor_SMD:C_0402_1005Metric -> Capacitor_SMD:C_1206_3216Metric
- C82, C83, C84: footprint Capacitor_SMD:C_0603_1608Metric -> Capacitor_SMD:C_1206_3216Metric
- J10, J11, J12, J13, J14, J15, J16, J2, J6, J7, J8, J9: value AFBR-2624Z -> HFBR-2521Z
- R1, R10, R11, R12, R13, R14, R15, R16, R17, R18, R19, R2, R20, R21, R22, R23, R24, R25, R26, R27, R28, R29, R3, R30, R31, R32, R33, R34, R35, R36, R37, R38, R39, R4, R40, R41, R42, R43, R44, R45, R46, R47, R48, R49, R5, R50, R51, R52, R53, R54, R55, R56, R57, R58, R59, R6, R60, R61, R62, R7, R8, R9: footprint Resistor_SMD:R_0603_1608Metric -> Resistor_SMD:R_1206_3216Metric
- moved C1 32.8 mm to (105.3, 51.2)
- moved C2 32.4 mm to (121.2, 51.0)
- moved C4 31.3 mm to (136.9, 50.8)
- moved C6 31.1 mm to (152.4, 50.6)
- moved C9 31.0 mm to (168.1, 50.8)
- moved C3 30.2 mm to (88.7, 51.2), turned to 180 degrees
- moved C5 20.4 mm to (72.3, 51.3), turned to 180 degrees
- moved C45 17.1 mm to (191.8, 105.8)
- moved C29 17.0 mm to (192.4, 75.0)
- moved C67 16.9 mm to (123.4, 135.2)
- moved C13 16.8 mm to (260.2, 75.6)
- moved C69 16.8 mm to (260.4, 165.8)
- moved C65 16.7 mm to (191.8, 135.7)
- moved C51 16.6 mm to (260.3, 135.7)
- moved C81 16.4 mm to (124.6, 165.2)
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Connections:
- J10 pad 1: Net-(J10-Data_Out) -> Net-(J10-Data_Out-Pad1)
- J10 pad 4: unconnected-(J10-NC-Pad4) -> Net-(J10-Data_Out-Pad1)
- J10 pad 5: GND -> unconnected-(J10-NC-Pad5)
- J10 pad 8: GND -> unconnected-(J10-NC-Pad8)
- J11 pad 1: Net-(J11-Data_Out) -> Net-(J11-Data_Out-Pad1)
- J11 pad 4: unconnected-(J11-NC-Pad4) -> Net-(J11-Data_Out-Pad1)
- J11 pad 5: GND -> unconnected-(J11-NC-Pad5)
- J11 pad 8: GND -> unconnected-(J11-NC-Pad8)
- J12 pad 1: Net-(J12-Data_Out) -> Net-(J12-Data_Out-Pad1)
- J12 pad 4: unconnected-(J12-NC-Pad4) -> Net-(J12-Data_Out-Pad1)
- J12 pad 5: GND -> unconnected-(J12-NC-Pad5)
- J12 pad 8: GND -> unconnected-(J12-NC-Pad8)
- J13 pad 1: Net-(J13-Data_Out) -> Net-(J13-Data_Out-Pad1)
- J13 pad 4: unconnected-(J13-NC-Pad4) -> Net-(J13-Data_Out-Pad1)
- J13 pad 5: GND -> unconnected-(J13-NC-Pad5)
- J13 pad 8: GND -> unconnected-(J13-NC-Pad8)
- J14 pad 1: Net-(J14-Data_Out) -> Net-(J14-Data_Out-Pad1)
- J14 pad 4: unconnected-(J14-NC-Pad4) -> Net-(J14-Data_Out-Pad1)
- J14 pad 5: GND -> unconnected-(J14-NC-Pad5)
- J14 pad 8: GND -> unconnected-(J14-NC-Pad8)
- J15 pad 1: Net-(J15-Data_Out) -> Net-(J15-Data_Out-Pad1)
- J15 pad 4: unconnected-(J15-NC-Pad4) -> Net-(J15-Data_Out-Pad1)
- J15 pad 5: GND -> unconnected-(J15-NC-Pad5)
- J15 pad 8: GND -> unconnected-(J15-NC-Pad8)
- J16 pad 1: Net-(J16-Data_Out) -> Net-(J16-Data_Out-Pad1)
- J16 pad 4: unconnected-(J16-NC-Pad4) -> Net-(J16-Data_Out-Pad1)
- J16 pad 5: GND -> unconnected-(J16-NC-Pad5)
- J16 pad 8: GND -> unconnected-(J16-NC-Pad8)
- J2 pad 1: Net-(J2-Data_Out) -> Net-(J2-Data_Out-Pad1)
- J2 pad 4: unconnected-(J2-NC-Pad4) -> Net-(J2-Data_Out-Pad1)
- J2 pad 5: GND -> unconnected-(J2-NC-Pad5)
- J2 pad 8: GND -> unconnected-(J2-NC-Pad8)
- J6 pad 1: Net-(J6-Data_Out) -> Net-(J6-Data_Out-Pad1)
- J6 pad 4: unconnected-(J6-NC-Pad4) -> Net-(J6-Data_Out-Pad1)
- J6 pad 5: GND -> unconnected-(J6-NC-Pad5)
- J6 pad 8: GND -> unconnected-(J6-NC-Pad8)
- J7 pad 1: Net-(J7-Data_Out) -> Net-(J7-Data_Out-Pad1)
- J7 pad 4: unconnected-(J7-NC-Pad4) -> Net-(J7-Data_Out-Pad1)
- J7 pad 5: GND -> unconnected-(J7-NC-Pad5)
- J7 pad 8: GND -> unconnected-(J7-NC-Pad8)
- J8 pad 1: Net-(J8-Data_Out) -> Net-(J8-Data_Out-Pad1)
- J8 pad 4: unconnected-(J8-NC-Pad4) -> Net-(J8-Data_Out-Pad1)
- J8 pad 5: GND -> unconnected-(J8-NC-Pad5)
- J8 pad 8: GND -> unconnected-(J8-NC-Pad8)
- J9 pad 1: Net-(J9-Data_Out) -> Net-(J9-Data_Out-Pad1)
- J9 pad 4: unconnected-(J9-NC-Pad4) -> Net-(J9-Data_Out-Pad1)
- J9 pad 5: GND -> unconnected-(J9-NC-Pad5)
- J9 pad 8: GND -> unconnected-(J9-NC-Pad8)
- U1 pad 2: Net-(J7-Data_Out) -> Net-(J7-Data_Out-Pad1)
- U13 pad 2: Net-(J9-Data_Out) -> Net-(J9-Data_Out-Pad1)
- U14 pad 2: Net-(J8-Data_Out) -> Net-(J8-Data_Out-Pad1)
- U15 pad 2: Net-(J13-Data_Out) -> Net-(J13-Data_Out-Pad1)
- U22 pad 2: Net-(J12-Data_Out) -> Net-(J12-Data_Out-Pad1)
- U23 pad 2: Net-(J11-Data_Out) -> Net-(J11-Data_Out-Pad1)
- U24 pad 2: Net-(J16-Data_Out) -> Net-(J16-Data_Out-Pad1)
- U31 pad 2: Net-(J15-Data_Out) -> Net-(J15-Data_Out-Pad1)
- U32 pad 2: Net-(J14-Data_Out) -> Net-(J14-Data_Out-Pad1)
- U4 pad 2: Net-(J2-Data_Out) -> Net-(J2-Data_Out-Pad1)
- U5 pad 2: Net-(J6-Data_Out) -> Net-(J6-Data_Out-Pad1)
- U6 pad 2: Net-(J10-Data_Out) -> Net-(J10-Data_Out-Pad1)
Routing:
- net Net-(J15-Data_Out-Pad1): track 0.00 -> 147.4 mm, vias 0 -> 1
- net Net-(J16-Data_Out-Pad1): track 0.00 -> 143.9 mm, vias 0 -> 1
- net Net-(J14-Data_Out-Pad1): track 0.00 -> 137.9 mm, vias 0 -> 1
- net Net-(J15-Data_Out): track 136.8 -> 0.00 mm, vias 1 -> 0
- net Net-(J16-Data_Out): track 136.4 -> 0.00 mm, vias 1 -> 0
- net Net-(J14-Data_Out): track 131.8 -> 0.00 mm, vias 1 -> 0
- net Net-(J13-Data_Out-Pad1): track 0.00 -> 109.2 mm, vias 0 -> 1
- net Net-(J12-Data_Out-Pad1): track 0.00 -> 104.0 mm, vias 0 -> 1
- net Net-(J11-Data_Out-Pad1): track 0.00 -> 101.2 mm, vias 0 -> 1
- net Net-(J13-Data_Out): track 99.8 -> 0.00 mm, vias 1 -> 0
- net Net-(J12-Data_Out): track 97.9 -> 0.00 mm, vias 1 -> 0
- net Net-(J11-Data_Out): track 95.0 -> 0.00 mm, vias 1 -> 0
- net Net-(J10-Data_Out-Pad1): track 0.00 -> 72.6 mm, vias 0 -> 1
- net Net-(J9-Data_Out-Pad1): track 0.00 -> 70.0 mm, vias 0 -> 1
- net Net-(J8-Data_Out-Pad1): track 0.00 -> 66.9 mm, vias 0 -> 1
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
Commit message: Completed Version 1: replace bury vias to micro vias
Routing:
- net ia_signal: track 162.3 -> 160.8 mm, vias 2 -> 1
- net GND: track 140.8 -> 141.4 mm
- net -BATT: vias 74 -> 70
- net +BATT: vias 60 -> 56
