File: Control_Board_Peripherals/Control_Board_Peripherals.kicad_pcb (KiCad board)
At the start: 2 copper layers, 192.5 x 122.4 mm, 94 parts, among them J10 HFBR-1521Z, J11 HFBR-1521Z, J12 HFBR-1521Z, J13 1827907, J14 HFBR-1521Z, J15 HFBR-1521Z, J16 HFBR-1521Z, J17 HFBR-1521Z, J18 HFBR-1521Z, J19 HFBR-1521Z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

Commit message: CCS project is added, PCB layout are updated, simulations are combined into one file, the completed version of c-script simulation is to be done.
Parts:
- added J1: 1714971, FYP_Components:CONN_1714971_PXC, F.Cu at (41.8, 140.4)
- added J3: 1714971, FYP_Components:CONN_1714971_PXC, F.Cu at (63.4, 140.4)
- added R40: 120k, Resistor_SMD:R_1206_3216Metric, F.Cu at (43.1, 133.4)
- added R41: 1k, Resistor_SMD:R_1206_3216Metric, F.Cu at (50.2, 133.4)
- added R42: 1k, Resistor_SMD:R_1206_3216Metric, F.Cu at (59.7, 133.2)
- added R43: 120k, Resistor_SMD:R_1206_3216Metric, F.Cu at (64.7, 133.2)
Connections:
- J2 pad 19: /ic_adc -> unconnected-(J2-Pin_19-Pad19)
- J2 pad 2: /ia_adc -> /ib_adc
- J2 pad 20: unconnected-(J2-Pin_20-Pad20) -> /ic_adc
- J2 pad 4: unconnected-(J2-Pin_4-Pad4) -> /ia_adc
- J2 pad 6: unconnected-(J2-Pin_6-Pad6) -> /sample_2
- J2 pad 8: unconnected-(J2-Pin_8-Pad8) -> /sample_1
- J2 pad 9: /ib_adc -> unconnected-(J2-Pin_9-Pad9)
Routing:
- net /sample_1: track 0.00 -> 62.9 mm
- net /sample_2: track 0.00 -> 46.1 mm
- net GND: track 203.2 -> 220.1 mm
- net -BATT: track 0.00 -> 9.78 mm
- net +BATT: track 0.00 -> 6.99 mm
- net /ia_adc: track 19.2 -> 23.9 mm
- net /ic_adc: track 9.94 -> 14.2 mm
- net /ib_adc: track 12.1 -> 15.7 mm
Other:
- board text added: "5V"
- board text added: "A"
- board text added: "A1"
- board text added: "A2"
- board text added: "A3"
- board text added: "A4"
- board text added: "B"
- board text added: "B1"
- board text added: "B2"
- board text added: "B3"
- board text added: "B4"
- board text added: "BATT+"
- board text added: "BATT-"
- board text added: "C1"
- board text added: "C2"
- board text added: "C3"
- board text added: "C4"
- board text added: "GND"
- board text added: "Index"
- board text added: "RX"
- board text added: "ia"
- board text added: "ib"
- board text added: "ic"
