File: Control_Board_Peripherals/Control_Board_Peripherals.kicad_sch (KiCad schematic)
At the start: 91 parts, among them J1 Conn_01x10_Pin, J2 Conn_01x10_Pin, J3 Conn_01x10_Pin, J4 1714971, J4 Conn_01x10_Pin, J5 1827907, J5 Conn_01x10_Pin, J6 Conn_01x10_Pin, J7 Conn_01x10_Pin, J8 Conn_01x10_Pin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

Commit message: Control board PCB layout is completed.
Parts:
- removed J1, J2, J3, J4, J5, J6, J7, J8: Conn_01x10_Pin, Connector_PinHeader_2.54mm:PinHeader_1x10_P2.54mm_Vertical, symbol Connector:Conn_01x10_Pin
- added C18, C19, C20, C21, C22: 0.1u, Capacitor_SMD:C_1206_3216Metric, symbol Device:C_Polarized
- added J2, J4, J5, J6: Conn_02x10_Top_Bottom, Connector_PinHeader_2.54mm:PinHeader_2x10_P2.54mm_Vertical, symbol Connector_Generic:Conn_02x10_Top_Bottom
- added J23: Conn_01x03, FYP_Components:CONN_1776511, symbol Connector_Generic:Conn_01x03
- added J24: Conn_01x05, FYP_Components:CONN_1827897, symbol Connector_Generic:Conn_01x05
- C1, C2, C3, C4, C5: value C_Polarized -> 0.1u; footprint (none) -> Capacitor_SMD:C_1206_3216Metric
- C10, C11, C12, C13, C14, C15, C16, C17, C6, C7, C8, C9: value C_Polarized -> 4.7u
- J10, J11, J12, J14, J15, J16, J17, J18, J19, J20, J21, J22: value ~ -> HFBR-1521Z
- R1, R11, R12, R13, R14, R15, R16, R2, R22, R23, R24, R25, R27, R28, R3, R34, R35, R36, R37, R38, R39, R4, R5, R6: value R -> 100
- R10, R29, R31: value R -> 10k
- R17, R32, R33: value R -> 330
- R18, R20, R7: value R -> 5.6k
- R19, R21, R8: value R -> 20k
- R26, R30, R9: value R -> 4.3k
- U1, U2, U3, U4, U5, U6: footprint D0008A_N -> FYP_Components:SN75451BD
Connections:
- net A1: now also J5.14 (Pin_14)
- net A2: now also J5.16 (Pin_16)
- net A3: now also J5.18 (Pin_18)
- net A4: now also J5.20 (Pin_20)
- net B1: now also J4.16 (Pin_16)
- net B2: now also J4.18 (Pin_18)
- net B3: now also J5.1 (Pin_1)
- net B4: now also J5.2 (Pin_2)
- net C1: now also J4.1 (Pin_1)
- net C2: now also J4.2 (Pin_2)
- net C3: now also J4.4 (Pin_4)
- net C4: now also J4.6 (Pin_6)
- net GND: now also J5.2, J5.4, J5.6, C18.2, C19.2, C20.2, C21.2, C22.2, J2.12 (Pin_12), J23.3 (Pin_3), J24.2 (Pin_2), J6.12 (Pin_12); no longer J5.1, J5.3, J5.5
- net SCIC_RX: now also J23.2 (Pin_2), J6.5 (Pin_5)
- net VCC: now also J2.11 (Pin_11), J23.1 (Pin_1), J24.1 (Pin_1), J6.11 (Pin_11)
- net ia_adc: now also J2.2 (Pin_2)
- net ia_signal: now also J5.1; no longer J5.2
- net ib_adc: now also J2.9 (Pin_9)
- net ib_signal: now also J5.3; no longer J5.4
- net ic_adc: now also J2.19 (Pin_19)
- net ic_signal: now also J5.5; no longer J5.6
- net +3.3VA renamed +3.3V
- net +3.3V: now also C18.1, C19.1, C20.1, C21.1, C22.1, J2.1 (Pin_1), J6.1 (Pin_1)
- new net CH_A: J24.3 (Pin_3), J6.15 (Pin_15)
- new net CH_B: J24.4 (Pin_4), J6.17 (Pin_17)
- new net Index: J24.5 (Pin_5), J6.19 (Pin_19)
- no-connect marks 51 -> 54
Other:
- note added: "Feedback Connectors"
- moved on the sheet: C1, C10, C11, C12, C13, C14, C15, C16, C17, C2, C3, C4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

Commit message: CCS project is added, PCB layout are updated, simulations are combined into one file, the completed version of c-script simulation is to be done.
Parts:
- added J4 (x2): 1714971, CONN_1714971_PXC, symbol FYP_Components:1714971
- added R40, R43: 120k, Resistor_SMD:R_1206_3216Metric, symbol Device:R
- added R41, R42: 1k, Resistor_SMD:R_1206_3216Metric, symbol Device:R
Connections:
- net GND: now also J4.1, J4.2, R41.2, R42.1
- net ia_adc: now also J2.4 (Pin_4); no longer J2.2 (Pin_2)
- net ib_adc: now also J2.2 (Pin_2); no longer J2.9 (Pin_9)
- net ic_adc: now also J2.20 (Pin_20); no longer J2.19 (Pin_19)
- net sample_2: now reaches J2.6 (Pin_6)
- net sample_2: now also R42.2, R43.1
- net sample_1: now reaches J2.8 (Pin_8)
- net sample_1: now also R40.2, R41.1
- new net +BATT: J4.1, R40.1
- new net -BATT: J4.2, R43.2
- no-connect marks 54 -> 53
Other:
- note removed: "5V Supply"
- note removed: "Current Signal Input"
- note removed: "Feedback Connectors"
- moved on the sheet: C1, C10, C11, C12, C13, C14, C15, C16, C17, C18, C19, C2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
