File: Control_Board_Peripherals/Control_Board_Peripherals.kicad_sch (KiCad schematic)
At the start: 101 parts, among them J10 HFBR-1521Z, J11 HFBR-1521Z, J12 HFBR-1521Z, J14 HFBR-1521Z, J15 HFBR-1521Z, J16 HFBR-1521Z, J17 HFBR-1521Z, J18 HFBR-1521Z, J19 HFBR-1521Z, J2 Conn_02x10_Top_Bottom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

Commit message: updated thesis: 8th May
Other:
- note added: "DC Voltage Sampling"
- note added: "Phase A Current Sampling"
Changed lines of the file:
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@@
     (stroke (width 0) (type default))
+  )
+  (text "DC Voltage Sampling" (at 98.552 111.252 0)
+    (effects (font (size 1.27 1.27)) (justify left bottom))
+  )
+  (text "Phase A Current Sampling" (at 195.8594 98.171 0)
+    (effects (font (size 1.27 1.27)) (justify left bottom))
   )
   (label "CH_B" (at 43.4594 90.5002 180) (fields_autoplaced)
